File: IOT_Board/IOT_Board.sch (KiCad schematic (older format))
At the start: 62 parts, among them Q1 2N3904, Q2 2N3904, Q3 2N3904, Q4 2N3904, Q5 2N3904, Q6 2N3904, x1 8M0, x2 32K768

Commit message: associated footprints, layed out PCB
Parts:
- removed C12, C9: 100p, symbol pspice:C
- removed C13, C14: 12p, symbol pspice:C
- removed C2, C4, C8: 100n, symbol pspice:C
- removed D13, D14: D_Zener_Small, symbol Device:D_Zener_Small
- removed D7, D8: blue, symbol Device:LED
- removed Q5, Q6: 2N3904, Package_TO_SOT_THT:TO-92_Inline, symbol Transistor_BJT:2N3904
- removed R21: 1k, symbol Device:R
- removed R22: 10k, symbol Device:R
- removed R23: 510r, symbol Device:R
- removed R3, R4: 100k, symbol Device:R
- removed Reset_sw1: SW_Push, symbol Switch:SW_Push
- removed boot_port1: Conn_02x03_Odd_Even, symbol Connector_Generic:Conn_02x03_Odd_Even
- removed debug_port1: Conn_01x04, symbol Connector_Generic:Conn_01x04
- removed mcu_1: STM32F103C8T6, Package_QFP:LQFP-48_7x7mm_P0.5mm, symbol MCU_ST_STM32F1:STM32F103C8Tx
- removed relay5, relay6: 5V_DC_Relay_Switch, symbol custom:5V_DC_Relay_Switch
- removed x1: 8M0, symbol Device:Crystal
- removed x2: 32K768, symbol Device:Crystal
- added Cin1: 10nf, Capacitor_THT:CP_Radial_D4.0mm_P1.50mm, symbol pspice:C
- added Cout1: 10uf, Capacitor_THT:CP_Radial_D4.0mm_P1.50mm, symbol pspice:C
- added D1: D_Zener_Small, Diode_THT:D_A-405_P7.62mm_Horizontal, symbol Device:D_Zener_Small
- added DCjack1: Barrel_Jack_Switch, Connector_BarrelJack:BarrelJack_Horizontal, symbol Connector:Barrel_Jack_Switch
- added J1, J2, J5, J6, J8: Screw_Terminal_01x03, TerminalBlock_4Ucon:TerminalBlock_4Ucon_1x03_P3.50mm_Horizontal, symbol Connector:Screw_Terminal_01x03
- added J10: Conn_02x04_Counter_Clockwise, Connector_PinHeader_1.00mm:PinHeader_2x04_P1.00mm_Vertical, symbol Connector_Generic:Conn_02x04_Counter_Clockwise
- added J3, J4: Conn_02x10_Counter_Clockwise, Connector_PinHeader_1.00mm:PinHeader_2x10_P1.00mm_Vertical, symbol Connector_Generic:Conn_02x10_Counter_Clockwise
- added J7: Screw_Terminal_01x05, TerminalBlock_4Ucon:TerminalBlock_4Ucon_1x05_P3.50mm_Horizontal, symbol Connector:Screw_Terminal_01x05
- added J9: Screw_Terminal_01x04, TerminalBlock_4Ucon:TerminalBlock_4Ucon_1x04_P3.50mm_Horizontal, symbol Connector:Screw_Terminal_01x04
- added Q1: 2N3904, Package_TO_SOT_THT:TO-92_Inline, symbol Transistor_BJT:2N3904
- added R1: 1k, Resistor_THT:R_Axial_DIN0204_L3.6mm_D1.6mm_P5.08mm_Horizontal, symbol Device:R
- added R17: 10k, Resistor_THT:R_Axial_DIN0204_L3.6mm_D1.6mm_P5.08mm_Horizontal, symbol Device:R
- added SW1, SW2: SW_Push, Button_Switch_THT:SW_PUSH_6mm_H13mm, symbol Switch:SW_Push
- added reg1: LD1117S33TR_SOT223, Package_TO_SOT_THT:TO-3P-3_Vertical, symbol Regulator_Linear:LD1117S33TR_SOT223
- added relay1: 5V_DC_Relay_Switch, Relay_THT:Relay_SPDT_SANYOU_SRD_Series_Form_C, symbol IOT_Board-rescue:5V_DC_Relay_Switch-custom
- D10: footprint (none) -> Diode_THT:D_A-405_P7.62mm_Horizontal
- D11: renamed from D4; footprint (none) -> LED_THT:LED_D3.0mm
- D2: footprint (none) -> LED_THT:LED_D3.0mm
- D3: renamed from D11; footprint (none) -> Diode_THT:D_A-405_P7.62mm_Horizontal
- D4: renamed from D5; footprint (none) -> LED_THT:LED_D3.0mm
- D5: renamed from D1; value red -> on; footprint (none) -> LED_THT:LED_D3.0mm
- D6: renamed from D12; footprint (none) -> Diode_THT:D_A-405_P7.62mm_Horizontal
- D7: renamed from D6; footprint (none) -> LED_THT:LED_D3.0mm
- D8: renamed from D9; footprint (none) -> Diode_THT:D_A-405_P7.62mm_Horizontal
- D9: renamed from D3; footprint (none) -> LED_THT:LED_D3.0mm
- R10: renamed from R6; footprint (none) -> Resistor_THT:R_Axial_DIN0204_L3.6mm_D1.6mm_P5.08mm_Horizontal
- R11: renamed from R7; footprint (none) -> Resistor_THT:R_Axial_DIN0204_L3.6mm_D1.6mm_P5.08mm_Horizontal
- R12: renamed from R17; footprint (none) -> Resistor_THT:R_Axial_DIN0204_L3.6mm_D1.6mm_P5.08mm_Horizontal
- R13: renamed from R8; footprint (none) -> Resistor_THT:R_Axial_DIN0204_L3.6mm_D1.6mm_P5.08mm_Horizontal
- R14: renamed from R9; footprint (none) -> Resistor_THT:R_Axial_DIN0204_L3.6mm_D1.6mm_P5.08mm_Horizontal
- R15: renamed from R10; footprint (none) -> Resistor_THT:R_Axial_DIN0204_L3.6mm_D1.6mm_P5.08mm_Horizontal
- R16: renamed from R11; footprint (none) -> Resistor_THT:R_Axial_DIN0204_L3.6mm_D1.6mm_P5.08mm_Horizontal
- R18: value 1k -> 470r; footprint (none) -> Resistor_THT:R_Axial_DIN0204_L3.6mm_D1.6mm_P5.08mm_Horizontal
- R19, R2, R5: footprint (none) -> Resistor_THT:R_Axial_DIN0204_L3.6mm_D1.6mm_P5.08mm_Horizontal
- R20: value 510r -> 10k; footprint (none) -> Resistor_THT:R_Axial_DIN0204_L3.6mm_D1.6mm_P5.08mm_Horizontal
- R3: renamed from R12; footprint (none) -> Resistor_THT:R_Axial_DIN0204_L3.6mm_D1.6mm_P5.08mm_Horizontal
- R4: renamed from R13; footprint (none) -> Resistor_THT:R_Axial_DIN0204_L3.6mm_D1.6mm_P5.08mm_Horizontal
- R6: renamed from R14; footprint (none) -> Resistor_THT:R_Axial_DIN0204_L3.6mm_D1.6mm_P5.08mm_Horizontal
- R7: renamed from R1; footprint (none) -> Resistor_THT:R_Axial_DIN0204_L3.6mm_D1.6mm_P5.08mm_Horizontal
- R8: renamed from R15; footprint (none) -> Resistor_THT:R_Axial_DIN0204_L3.6mm_D1.6mm_P5.08mm_Horizontal
- R9: renamed from R16; footprint (none) -> Resistor_THT:R_Axial_DIN0204_L3.6mm_D1.6mm_P5.08mm_Horizontal
- relay2: renamed from relay3; footprint (none) -> Relay_THT:Relay_SPDT_SANYOU_SRD_Series_Form_C; symbol custom:5V_DC_Relay_Switch -> IOT_Board-rescue:5V_DC_Relay_Switch-custom
- relay3: renamed from relay4; footprint (none) -> Relay_THT:Relay_SPDT_SANYOU_SRD_Series_Form_C; symbol custom:5V_DC_Relay_Switch -> IOT_Board-rescue:5V_DC_Relay_Switch-custom
- relay4: renamed from relay1; footprint (none) -> Relay_THT:Relay_SPDT_SANYOU_SRD_Series_Form_C; symbol custom:5V_DC_Relay_Switch -> IOT_Board-rescue:5V_DC_Relay_Switch-custom
- relay5: renamed from relay2; footprint (none) -> Relay_THT:Relay_SPDT_SANYOU_SRD_Series_Form_C; symbol custom:5V_DC_Relay_Switch -> IOT_Board-rescue:5V_DC_Relay_Switch-custom
- renumbered Q3 to Q2, Q4 to Q3, Q1 to Q4, Q2 to Q5
Connections:
- net reset is gone; now on net GND: R2.2
- net s5 is gone; now on net GND: R18.2
- net GND: now also D2.1 (K), Cin1.2, Cout1.2, DCjack1.2, DCjack1.3, J10.1 (Pin_1), J3.19 (Pin_19), J4.20 (Pin_20), SW2.1, reg1.1 (GND); no longer R19.2
- net s1: now also J4.18 (Pin_18)
- net s2: now also J3.2 (Pin_2)
- net s3: now also J3.5 (Pin_5)
- net s4: now also J3.6 (Pin_6)
- net at R5.1: now also Q1.1 (E); no longer D2.1 (K)
- net at D8.2 (A), Q4.3 (C): now also relay4.2 (gnd); no longer relay4.~ (5)
- net at D10.2 (A), Q5.3 (C): now also relay5.2 (gnd); no longer relay5.~ (5)
- net at D3.2 (A), Q2.3 (C): now also relay2.2 (gnd); no longer relay2.~ (5)
- net vcc3v3: now reaches R20.1
- net vcc3v3: now also R19.1, Cout1.1, J10.5 (Pin_5), J3.1 (Pin_1), R17.1, reg1.2 (VO)
- net at R18.1: now also SW1.1; no longer R19.1
- net en: now reaches R20.2
- net en: now also J10.7 (Pin_7)
- net at D6.2 (A), Q3.3 (C): now also relay3.2 (gnd); no longer relay3.~ (5)
- removed net +3V3: D2.2 (A), D5.2 (A), R2.1
- net +5V renamed vcc5v
- net vcc5v: now also D5.2 (A), relay2.5 (vcc), relay3.5 (vcc), relay4.5 (vcc), relay5.5 (vcc), Cin1.1, D1.1 (K), DCjack1.1, J3.20 (Pin_20), reg1.3 (VI), relay1.5 (vcc); no longer relay2.~ (5), relay3.~ (5), relay4.~ (5), relay5.~ (5)
- net pc13: no longer names the net of R5.2
- net pc13: now also D2.2 (A)
- new net: J6.2 (Pin_2), relay4.1 (C)
- new net: J6.1 (Pin_1), relay4.3 (NO)
- new net: J6.3 (Pin_3), relay4.4 (NC)
- new net: J8.2 (Pin_2), relay5.1 (C)
- new net: J8.1 (Pin_1), relay5.3 (NO)
- new net: J8.3 (Pin_3), relay5.4 (NC)
- new net: J2.2 (Pin_2), relay2.1 (C)
- new net: J2.1 (Pin_1), relay2.3 (NO)
- new net: J2.3 (Pin_3), relay2.4 (NC)
- new net: J5.2 (Pin_2), relay3.1 (C)
- new net: J5.1 (Pin_1), relay3.3 (NO)
- new net: J5.3 (Pin_3), relay3.4 (NC)
- new net: Q1.2 (B), R1.1, R2.1
- new net: D1.2 (A), Q1.3 (C), relay1.2 (gnd)
- new net: J1.2 (Pin_2), relay1.1 (C)
- new net: J1.1 (Pin_1), relay1.3 (NO)
- new net: J1.3 (Pin_3), relay1.4 (NC)
- new net an0: J3.12 (Pin_12), J9.1 (Pin_1)
- new net an1: J3.13 (Pin_13), J9.2 (Pin_2)
- new net an10: J3.7 (Pin_7), J9.4 (Pin_4)
- new net an2: J3.14 (Pin_14), J9.3 (Pin_3)
- new net ch0: J4.13 (Pin_13), J7.1 (Pin_1)
- new net ch1: J3.18 (Pin_18), J7.2 (Pin_2)
- new net ch2: J3.17 (Pin_17), J7.3 (Pin_3)
- new net ch3: J3.16 (Pin_16), J7.4 (Pin_4)
- new net ch4: J3.15 (Pin_15), J7.5 (Pin_5)
- new net io0: J10.3 (Pin_3), R17.2, SW1.2
- new net rs: J10.6 (Pin_6), R19.2, SW2.2
- new net rx: J10.4 (Pin_4), J3.4 (Pin_4)
- new net s0: J4.19 (Pin_19), J4.8 (Pin_8), R1.2
- new net tx: J10.8 (Pin_8), J3.3 (Pin_3)
Other:
- moved on the sheet: D10, D11, D3, D4, D5, D6, D7, D8, D9, Q2, Q3, Q4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
